Commit message: 完成了基本的显示/轨迹规划

File: src/robotic_arm/urdf/robotic_arm.urdf (robot description, URDF)
Before this commit: robot robotic_arm, 7 links, 6 joints
Joints:
- joint joint1: origin xyz=0 1.09157351461941E-05 0.0566 rpy=0 0 0 -> xyz=0 1.09157351461941E-05 0.0566 rpy=0 0 0.0
- joint joint2: origin xyz=0 -0.121299999999996 0.118000000000003 rpy=-1.5707963267949 -1.22156142621659 0 -> xyz=0 -0.121299999999996 0.118000000000003 rpy=-1.5707963267949 -1.5707963267949 0
- joint joint3: origin xyz=0.555000000000002 0 0.0804999999999991 rpy=0 0 2.05967901546526 -> xyz=0.555000000000002 0 0.0804999999999991 rpy=0 0 0
- joint joint4: origin xyz=0.535949999999994 0 -0.0276499999999935 rpy=0 0 -0.855870532287509 -> xyz=0.535949999999994 0 -0.0276499999999935 rpy=0 0 0

File: src/robotic_config/config/robotic_arm.ros2_control.xacro (robot description, xacro)
@@ -10,61 +10,43 @@
             <joint name="joint1">
                 <command_interface name="position"/>
-                <command_interface name="velocity"/>
-                <command_interface name="effort"/>
                 <state_interface name="position">
                   <param name="initial_value">${initial_positions['joint1']}</param>
                 </state_interface>
                 <state_interface name="velocity"/>
-                <state_interface name="effort"/>
             </joint>
             <joint name="joint2">
                 <command_interface name="position"/>
-                <command_interface name="velocity"/>
-                <command_interface name="effort"/>
                 <state_interface name="position">
                   <param name="initial_value">${initial_positions['joint2']}</param>
                 </state_interface>
                 <state_interface name="velocity"/>
-                <state_interface name="effort"/>
             </joint>
             <joint name="joint3">
                 <command_interface name="position"/>
-                <command_interface name="velocity"/>
-                <command_interface name="effort"/>
                 <state_interface name="position">
                   <param name="initial_value">${initial_positions['joint3']}</param>
                 </state_interface>
                 <state_interface name="velocity"/>
-                <state_interface name="effort"/>
             </joint>
             <joint name="joint4">
                 <command_interface name="position"/>
-                <command_interface name="velocity"/>
-                <command_interface name="effort"/>
                 <state_interface name="position">
                   <param name="initial_value">${initial_positions['joint4']}</param>
                 </state_interface>
                 <state_interface name="velocity"/>
-                <state_interface name="effort"/>
             </joint>
             <joint name="joint5">
                 <command_interface name="position"/>
-                <command_interface name="velocity"/>
-                <command_interface name="effort"/>
                 <state_interface name="position">
                   <param name="initial_value">${initial_positions['joint5']}</param>
                 </state_interface>
                 <state_interface name="velocity"/>
-                <state_interface name="effort"/>
             </joint>
             <joint name="joint6">
                 <command_interface name="position"/>
-                <command_interface name="velocity"/>
-                <command_interface name="effort"/>
                 <state_interface name="position">
                   <param name="initial_value">${initial_positions['joint6']}</param>
                 </state_interface>
                 <state_interface name="velocity"/>
-                <state_interface name="effort"/>
             </joint>
         </ros2_control>

Commit message: 实现了机械臂位置在理论上的实时更新

File: src/robotic_arm/urdf/robotic_arm.urdf (robot description, URDF)
Before this commit: robot robotic_arm, 7 links, 6 joints
Links:
- link base_link: mass 0.450435332011656 -> None

Commit message: 完成了仿真环境下的机械臂抓取KFS并放置，然后恢复到空闲姿态的完整动作

File: src/robotic_arm/urdf/robotic_arm.urdf (robot description, URDF)
Before this commit: robot robotic_arm, 7 links, 6 joints
Joints:
- joint joint2: limit lower=-3.14159 upper=3.14159 effort=50 velocity=10 -> lower=-1.47 upper=1.47 effort=50 velocity=10

Commit message: 完成了对物理机械臂的基本操控，基本实现了取KFS，放KFS动作流程

File: src/robotic_arm/urdf/robotic_arm.urdf (robot description, URDF)
Before this commit: robot robotic_arm, 7 links, 6 joints
Joints:
- joint joint1: limit lower=-3.14159 upper=3.14159 effort=50 velocity=10 -> lower=-1.47 upper=1.47 effort=50 velocity=10

Commit message: 新机械臂

File: src/robotic_arm/urdf/robotic_arm.urdf (robot description, URDF)
Before this commit: robot robotic_arm, 7 links, 6 joints
Links:
- link base_link: mass None -> 1.0998
- link link1: mass 1.58241928661162 -> 2.36887473210498
- link link2: mass 2.73444383071047 -> 1.26008517135461
- link link3: mass 2.26799555337397 -> 0.384351971964209
- link link4: mass 0.196984301264057 -> 1.54177209175348
- link link5: mass 0.0669824634679072 -> 0.0662052566611412
- link link6: mass 0.145741627039506 -> 0.128099358994803
Joints:
- joint joint1: axis 0 0 -1 -> 0 0 1; limit lower=-1.47 upper=1.47 effort=50 velocity=10 -> lower=0 upper=0 effort=0 velocity=0; origin xyz=0 1.09157351461941E-05 0.0566 rpy=0 0 0.0 -> xyz=0 0 0 rpy=0 0 0
- joint joint2: axis 0 0 -1 -> 0 0 1; limit lower=-1.47 upper=1.47 effort=50 velocity=10 -> lower=0 upper=0 effort=0 velocity=0; origin xyz=0 -0.121299999999996 0.118000000000003 rpy=-1.5707963267949 -1.5707963267949 0 -> xyz=0 0.03675 0.153 rpy=1.5708 -1.1673 0
- joint joint3: limit lower=-3.14159 upper=3.14159 effort=50 velocity=10 -> lower=0 upper=0 effort=0 velocity=0; origin xyz=0.555000000000002 0 0.0804999999999991 rpy=0 0 0 -> xyz=0.52 0 0.08565 rpy=0 0 -2.6342
- joint joint4: axis 0 0 1 -> 0 0 -1; limit lower=-3.14159 upper=3.14159 effort=50 velocity=10 -> lower=0 upper=0 effort=0 velocity=0; origin xyz=0.535949999999994 0 -0.0276499999999935 rpy=0 0 0 -> xyz=0.436 0 0.0225 rpy=0 0 1.4725
- joint joint5: axis 0 0 -1 -> -1 0 0; limit lower=-3.14159 upper=3.14159 effort=50 velocity=10 -> lower=0 upper=0 effort=0 velocity=0; origin xyz=0 0.0335000000001389 0.0663799999999916 rpy=1.5707963267949 0.0631517658353735 0 -> xyz=0.07761 -0.0058889 -0.03035 rpy=-1.5708 0 0
- joint joint6: limit lower=-3.14159 upper=3.14159 effort=50 velocity=10 -> lower=0 upper=0 effort=0 velocity=0; origin xyz=0.0585072463768114 0 0.03335 rpy=-2.02961305550173 1.57079631189374 1.11099364899658 -> xyz=0.073796 0.0036822 8.8922E-05 rpy=0.051163 -1.5708 0

Commit message: 最初

File: src/robotic_arm/urdf/robotic_arm.urdf (robot description, URDF)
Before this commit: robot robotic_arm, 7 links, 6 joints
Links:
- link base_link: mass 1.0998 -> None
- link link1: mass 2.36887473210498 -> 1.58241928661162
- link link2: mass 1.26008517135461 -> 2.73444383071047
- link link3: mass 0.384351971964209 -> 2.26799555337397
- link link4: mass 1.54177209175348 -> 0.196984301264057
- link link5: mass 0.0662052566611412 -> 0.0669824634679072
- link link6: mass 0.128099358994803 -> 0.145741627039506
Joints:
- joint joint1: axis 0 0 1 -> 0 0 -1; limit lower=0 upper=0 effort=0 velocity=0 -> lower=-1.47 upper=1.47 effort=50 velocity=10; origin xyz=0 0 0 rpy=0 0 0 -> xyz=0 1.09157351461941E-05 0.0566 rpy=0 0 0.0
- joint joint2: axis 0 0 1 -> 0 0 -1; limit lower=0 upper=0 effort=0 velocity=0 -> lower=-1.47 upper=1.47 effort=50 velocity=10; origin xyz=0 0.03675 0.153 rpy=1.5708 -1.1673 0 -> xyz=0 -0.121299999999996 0.118000000000003 rpy=-1.5707963267949 -1.5707963267949 0
- joint joint3: limit lower=0 upper=0 effort=0 velocity=0 -> lower=-3.14159 upper=3.14159 effort=50 velocity=10; origin xyz=0.52 0 0.08565 rpy=0 0 -2.6342 -> xyz=0.555000000000002 0 0.0804999999999991 rpy=0 0 0
- joint joint4: axis 0 0 -1 -> 0 0 1; limit lower=0 upper=0 effort=0 velocity=0 -> lower=-3.14159 upper=3.14159 effort=50 velocity=10; origin xyz=0.436 0 0.0225 rpy=0 0 1.4725 -> xyz=0.535949999999994 0 -0.0276499999999935 rpy=0 0 0
- joint joint5: axis -1 0 0 -> 0 0 -1; limit lower=0 upper=0 effort=0 velocity=0 -> lower=-3.14159 upper=3.14159 effort=50 velocity=10; origin xyz=0.07761 -0.0058889 -0.03035 rpy=-1.5708 0 0 -> xyz=0 0.0335000000001389 0.0663799999999916 rpy=1.5707963267949 0.0631517658353735 0
- joint joint6: limit lower=0 upper=0 effort=0 velocity=0 -> lower=-3.14159 upper=3.14159 effort=50 velocity=10; origin xyz=0.073796 0.0036822 8.8922E-05 rpy=0.051163 -1.5708 0 -> xyz=0.0585072463768114 0 0.03335 rpy=-2.02961305550173 1.57079631189374 1.11099364899658

Commit message: 3-19

File: src/robotic_arm/urdf/robotic_arm.urdf (robot description, URDF)
Before this commit: robot robotic_arm, 7 links, 6 joints
Joints:
- joint joint1: limit lower=-1.47 upper=1.47 effort=50 velocity=10 -> lower=-6.283185307 upper=6.283185307 effort=50 velocity=10
- joint joint2: limit lower=-1.134464014 upper=1.570796327 effort=50 velocity=10 -> lower=-1.570796327 upper=1.570796327 effort=50 velocity=10; origin xyz=0 0.03675 0.153 rpy=1.5708 -1.1579 0 -> xyz=0 0.03675 0.153 rpy=1.5708 -1.5708 0
- joint joint3: limit lower=0.0 upper=5.759586532 effort=50 velocity=10 -> lower=-3.141592654 upper=3.141592654 effort=50 velocity=10; origin xyz=0.52 0 0.08565 rpy=0 0 -2.7359 -> xyz=0.52 0 0.08565 rpy=0 0 0
- joint joint4: limit lower=-3.14159 upper=3.14159 effort=50 velocity=10 -> lower=-3.141592654 upper=3.141592654 effort=50 velocity=10; origin xyz=0.436 0 0.0225 rpy=0 0 1.5836 -> xyz=0.436 0 0.0225 rpy=0 0 0
- joint joint6: origin xyz=0.073796 0.0036822 8.8922E-05 rpy=0.051163 -1.5708 0 -> xyz=0.073796 0.0036822 8.8922E-05 rpy=0 -1.5708 0
